File: schematics/ISA_Card/KiCad_Project/ps2_mouse_to_serial_port_adapter_ISA_card.kicad_sch (KiCad schematic)
At the start: 17 parts, among them J1 Serial Port, J2 Mini-DIN-6, J3 Bus_ISA_8bit, Q1 BC547, U1 74LS00, U2 L78L05

Commit message: v1.4.0
- Pequeños ajustes al tamaño y contorno de la placa ISA.
- Se han añadido zonas de relleno para GND en la placa ISA.
- Sin cambios en el software.
- Importante! Recordad que aún no he podido verificar en "físico" el diseño de las placas, por lo que recomiendo precaución si van a ser usadas.
Connections:
- net +5V: now reaches A1.30 (VIN), C1.1, C2.1, J2.4, J3.3 (VCC), R3.1, R5.1, U1.14 (VCC)
- net GND: now reaches A1.29 (GND), C1.2, C2.2, D2.1 (K), D3.1 (K), J1.5 (Pin_5), J2.3, J3.1 (GND), Q1.3 (E), R2.2, U1.7 (GND), U2.2 (GND)
Changed lines of the file:
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@@
     (title "PS/2 Mouse to Serial Port Adapter")
     (date "2023-08-12")
-    (rev "3")
+    (rev "4")
     (company "Cesar Rincon")
     (comment 1 "NightFox & Co.")
@@
     (effects (font (size 1.27 1.27)) (justify left bottom))
   )
-  (text "+5V" (at 241.3 20.32 0)
-    (effects (font (size 1.27 1.27)) (justify left bottom))
-  )
   (text "RTS" (at 52.07 165.1 0)
     (effects (font (size 1.27 1.27)) (justify left bottom))
@@
   )
   (text "+5V" (at 38.1 77.47 90)
-    (effects (font (size 1.27 1.27)) (justify left bottom))
-  )
-  (text "GND" (at 152.4 185.42 0)
     (effects (font (size 1.27 1.27)) (justify left bottom))
   )
@@
     (effects (font (size 1.27 1.27)) (justify left bottom))
   )
+  (label "GND" (at 151.13 181.61 0) (fields_autoplaced)
+    (effects (font (size 1.27 1.27)) (justify left bottom))
+  )
+  (label "+5V" (at 264.16 22.86 0) (fields_autoplaced)
+    (effects (font (size 1.27 1.27)) (justify left bottom))
+  )

Commit message: v1.5.1
- Arreglada la serigrafía del conector MINI-DIN-6 (PS/2), la cual se superponía en algunas zonas de soldado.
- En todas las placas se añade el símbolo de los agujeros de montaje con el tamaño estándar M3.
Parts:
- added H1, H2: MountingHole, MountingHole:MountingHole_3.2mm_M3, symbol Mechanical:MountingHole
- J2: footprint CustomLib:Conn_Mini_DIN_6pin -> ProjectLibrary:Connector_Mini_DIN_6pin
- J3: footprint CustomLib:BUS_AT -> ProjectLibrary:BUS_AT_ISA_8BITS
Changed lines of the file:
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@@
   (title_block
     (title "PS/2 Mouse to Serial Port Adapter")
-    (date "2023-08-12")
-    (rev "4")
+    (date "2023-08-14")
+    (rev "5")
     (company "Cesar Rincon")
     (comment 1 "NightFox & Co.")
@@
       (effects (font (size 1.27 1.27)) (justify right))
     )
-    (property "Footprint" "CustomLib:BUS_AT" (at 62.23 36.83 0)
+    (property "Footprint" "ProjectLibrary:BUS_AT_ISA_8BITS" (at 62.23 36.83 0)
       (effects (font (size 1.27 1.27)) hide)
     )
@@
     )
   )
+  (symbol (lib_id "Mechanical:MountingHole") (at -120.65 48.26 0) (unit 1)
+    (in_bom yes) (on_board yes) (dnp no) (fields_autoplaced)
+    (property "Reference" "H1" (at -118.11 46.99 0)
+      (effects (font (size 1.27 1.27)) (justify left))
+    )
+    (property "Value" "MountingHole" (at -118.11 49.53 0)
+      (effects (font (size 1.27 1.27)) (justify left))
+    )
+    (property "Footprint" "MountingHole:MountingHole_3.2mm_M3" (at -120.65 48.26 0)
+      (effects (font (size 1.27 1.27)) hide)
+    )
+    (property "Datasheet" "~" (at -120.65 48.26 0)
+      (effects (font (size 1.27 1.27)) hide)
+    )
+    (instances
+      (project "ps2_mouse_to_serial_port_adapter_ISA_card"
+        (path "/a7ffaf24-5f7f-4c3c-9493-bf517f6435f3"
+          (reference "H1") (unit 1)
+        )
+      )
+    )
+  )
   (symbol (lib_id "74xx:74LS00") (at -118.11 22.86 0) (unit 4)
     (in_bom yes) (on_board yes) (dnp no) (fields_autoplaced)
@@
       (effects (font (size 1.27 1.27)))
     )
-    (property "Footprint" "CustomLib:Conn_Mini_DIN_6pin" (at 54.61 109.22 0)
+    (property "Footprint" "ProjectLibrary:Connector_Mini_DIN_6pin" (at 54.61 109.22 0)
       (effects (font (size 1.27 1.27)) hide)
     )
@@
         )
       )
+    )
+  )
+  (symbol (lib_id "Mechanical:MountingHole") (at -120.65 55.88 0) (unit 1)
+    (in_bom yes) (on_board yes) (dnp no) (fields_autoplaced)
+    (property "Reference" "H2" (at -118.11 54.61 0)
+      (effects (font (size 1.27 1.27)) (justify left))
+    )
+    (property "Value" "MountingHole" (at -118.11 57.15 0)
+      (effects (font (size 1.27 1.27)) (justify left))
+    )
+    (property "Footprint" "MountingHole:MountingHole_3.2mm_M3" (at -120.65 55.88 0)
+      (effects (font (size 1.27 1.27)) hide)
+    )
+    (property "Datasheet" "~" (at -120.65 55.88 0)
+      (effects (font (size 1.27 1.27)) hide)
+    )
+    (instances
+      (project "ps2_mouse_to_serial_port_adapter_ISA_card"
+        (path "/a7ffaf24-5f7f-4c3c-9493-bf517f6435f3"
+          (reference "H2") (unit 1)
+        )
+      )

Commit message: v1.7.0
- Modificadas las huellas de todas las placas para que los componentes TO92 resulten más fáciles de soldar a mano.
- Modificadas las conexiones del conector IDC en la placa ISA para poder usar un cable IDC a DB9 comercial, sin necesidad de realizarle modificaciones.
- Añadido el modelo en formato FreeCad y el archivo STL del soporte para la placa ISA. Estos archivos estan preparados para poder realizar la impresión en 3D del soporte. Se recomienda un in-fill del 100%.
Parts:
- J1: value Serial Port -> IDC Connector
- Q1, U2: footprint Package_TO_SOT_THT:TO-92_Inline -> Package_TO_SOT_THT:TO-92_HandSolder
Connections:
- net GND: now also J1.9 (Pin_9); no longer J1.5 (Pin_5)
- net at D1.2 (A): now also J1.4 (Pin_4); no longer J1.7 (Pin_7)
- net at U1.3: now also J1.3 (Pin_3); no longer J1.2 (Pin_2)
Other:
- note added: "[2]"
- note added: "[2] [5] [7] Pins on the DB9 of the serial port"
- note added: "[5]"
- note added: "[7]"
Changed lines of the file:
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@@
   (title_block
     (title "PS/2 Mouse to Serial Port Adapter")
-    (date "2023-08-14")
-    (rev "5")
+    (date "2023-08-28")
+    (rev "6")
     (company "Cesar Rincon")
     (comment 1 "NightFox & Co.")
@@
   (junction (at 95.25 137.16) (diameter 0) (color 0 0 0 0)
   )
+  (junction (at 24.13 172.72) (diameter 0) (color 0 0 0 0)
+  )
   (junction (at 133.35 181.61) (diameter 0) (color 0 0 0 0)
   )
@@
   (no_connect (at 92.71 54.61))
   (no_connect (at 49.53 154.94))
+  (no_connect (at 46.99 142.24))
   (no_connect (at 72.39 54.61))
   (no_connect (at -125.73 25.4))
@@
   (no_connect (at -125.73 20.32))
   (no_connect (at 90.17 19.05))
+  (no_connect (at 39.37 142.24))
   (no_connect (at 67.31 54.61))
   (no_connect (at 49.53 142.24))
@@
   (no_connect (at 203.2 93.98))
   (no_connect (at 228.6 93.98))
-  (no_connect (at 44.45 142.24))
   (no_connect (at 72.39 19.05))
   (no_connect (at 218.44 73.66))
@@
   (no_connect (at 74.93 19.05))
   (no_connect (at 62.23 54.61))
-  (no_connect (at 41.91 142.24))
   (no_connect (at 44.45 154.94))
   (no_connect (at 67.31 19.05))
@@
   (no_connect (at 34.29 19.05))
   (no_connect (at 228.6 106.68))
-  (no_connect (at 41.91 154.94))
   (no_connect (at 54.61 54.61))
   (no_connect (at 59.69 19.05))
@@
   (no_connect (at 203.2 99.06))
   (no_connect (at 49.53 19.05))
+  (no_connect (at 46.99 154.94))
   (no_connect (at 31.75 19.05))
   (no_connect (at 44.45 54.61))
@@
     (stroke (width 0) (type default))
   )
-  (wire (pts (xy 24.13 129.54) (xy 24.13 181.61))
-    (stroke (width 0) (type default))
-  )
   (wire (pts (xy 133.35 62.23) (xy 213.36 62.23))
     (stroke (width 0) (type default))
   )
+  (wire (pts (xy 41.91 154.94) (xy 41.91 172.72))
+    (stroke (width 0) (type default))
+  )
   (wire (pts (xy 110.49 161.29) (xy 118.11 161.29))
     (stroke (width 0) (type default))
@@
     (stroke (width 0) (type default))
   )
-  (wire (pts (xy 46.99 161.29) (xy 64.77 161.29))
-    (stroke (width 0) (type default))
-  )
-  (wire (pts (xy 46.99 154.94) (xy 46.99 161.29))
-    (stroke (width 0) (type default))
-  )
   (wire (pts (xy 69.85 106.68) (xy 69.85 88.9))
     (stroke (width 0) (type default))
   )
-  (wire (pts (xy 80.01 137.16) (xy 46.99 137.16))
+  (wire (pts (xy 44.45 137.16) (xy 80.01 137.16))
     (stroke (width 0) (type default))
   )
@@
     (stroke (width 0) (type default))
   )
-  (wire (pts (xy 46.99 137.16) (xy 46.99 142.24))
-    (stroke (width 0) (type default))
-  )
   (wire (pts (xy 62.23 109.22) (xy 69.85 109.22))
     (stroke (width 0) (type default))
@@
     (stroke (width 0) (type default))
   )
+  (wire (pts (xy 24.13 129.54) (xy 24.13 172.72))
+    (stroke (width 0) (type default))
+  )
   (wire (pts (xy 133.35 181.61) (xy 170.18 181.61))
     (stroke (width 0) (type default))
@@
     (stroke (width 0) (type default))
   )
+  (wire (pts (xy 41.91 172.72) (xy 24.13 172.72))
+    (stroke (width 0) (type default))
+  )
   (wire (pts (xy 227.33 50.8) (xy 227.33 57.15))
     (stroke (width 0) (type default))
@@
     (stroke (width 0) (type default))
   )
+  (wire (pts (xy 41.91 142.24) (xy 41.91 137.16))
+    (stroke (width 0) (type default))
+  )
   (wire (pts (xy 62.23 106.68) (xy 69.85 106.68))
     (stroke (width 0) (type default))
@@
     (stroke (width 0) (type default))
   )
+  (wire (pts (xy 31.75 137.16) (xy 31.75 161.29))
+    (stroke (width 0) (type default))
+  )
   (wire (pts (xy 157.48 86.36) (xy 203.2 86.36))
     (stroke (width 0) (type default))
@@
     (stroke (width 0) (type default))
   )
+  (wire (pts (xy 44.45 137.16) (xy 44.45 142.24))
+    (stroke (width 0) (type default))
+  )
   (wire (pts (xy 95.25 137.16) (xy 106.68 137.16))
     (stroke (width 0) (type default))
@@
     (stroke (width 0) (type default))
   )
+  (wire (pts (xy 41.91 137.16) (xy 31.75 137.16))
+    (stroke (width 0) (type default))
+  )
   (wire (pts (xy 218.44 149.86) (xy 264.16 149.86))
     (stroke (width 0) (type default))
@@
     (stroke (width 0) (type default))
   )
+  (wire (pts (xy 24.13 172.72) (xy 24.13 181.61))
+    (stroke (width 0) (type default))
+  )
   (wire (pts (xy 106.68 111.76) (xy 157.48 111.76))
     (stroke (width 0) (type default))
   )
-  (wire (pts (xy 39.37 129.54) (xy 39.37 142.24))
+  (wire (pts (xy 31.75 161.29) (xy 64.77 161.29))
     (stroke (width 0) (type default))
   )
@@
     (effects (font (size 1.27 1.27)) (justify left bottom))
   )
+  (text "[5]" (at 33.02 171.45 0)
+    (effects (font (size 1.27 1.27) bold) (justify left bottom))
+  )
   (text "GND" (at 267.97 105.41 90)
     (effects (font (size 1.27 1.27)) (justify left bottom))
   )
+  (text "[2]" (at 48.26 135.89 0)
+    (effects (font (size 1.27 1.27) (thickness 0.254) bold) (justify left bottom))
+  )
   (text "VCC +5V" (at 27.94 106.68 0)
     (effects (font (size 1.27 1.27)) (justify left bottom))
   )
+  (text "[2] [5] [7]\nPins on the DB9\nof the serial port" (at 45.72 171.45 0)
+    (effects (font (size 1.27 1.27) italic) (justify left bottom))
+  )
   (text "16V" (at 43.18 123.19 0)
     (effects (font (size 1.27 1.27)) (justify left bottom))
@@
     (effects (font (size 1.27 1.27)) (justify left bottom))
   )
-  (text "RTS" (at 52.07 165.1 0)
+  (text "RTS" (at 36.83 135.89 0)
     (effects (font (size 1.27 1.27)) (justify left bottom))
   )
@@
     (effects (font (size 1.27 1.27)) (justify left bottom))
   )
-  (text "GND" (at 21.59 154.94 90)
-    (effects (font (size 1.27 1.27)) (justify left bottom))
+  (text "GND" (at 40.64 171.45 0)
+    (effects (font (size 1.27 1.27)) (justify right bottom))
+  )
+  (text "[7]" (at 33.02 135.89 0)
+    (effects (font (size 1.27 1.27) bold) (justify left bottom))
   )
   (text "+DATA" (at 77.47 110.49 0)
@@
       (effects (font (size 1.27 1.27)) (justify left))
     )
-    (property "Footprint" "Package_TO_SOT_THT:TO-92_Inline" (at 135.89 163.195 0)
+    (property "Footprint" "Package_TO_SOT_THT:TO-92_HandSolder" (at 135.89 163.195 0)
       (effects (font (size 1.27 1.27) italic) (justify left) hide)
     )
@@
       (effects (font (size 1.27 1.27)))
     )
-    (property "Footprint" "Package_TO_SOT_THT:TO-92_Inline" (at 87.63 155.575 0)
+    (property "Footprint" "Package_TO_SOT_THT:TO-92_HandSolder" (at 87.63 155.575 0)
       (effects (font (size 1.27 1.27) italic) hide)
     )
@@
       (effects (font (size 1.27 1.27)) (justify left))
     )
-    (property "Value" "Serial Port" (at 52.07 149.86 90)
-      (effects (font (size 1.27 1.27)) (justify left))
-    )
+    (property "Value" "IDC Connector" (at 52.07 149.86 90)
+      (effects (font (size 1.27 1.27)) (justify left))
+    )
