File: schematics/ISA_Card/KiCad_Project/ps2_mouse_to_serial_port_adapter_ISA_card.kicad_pcb (KiCad board)
At the start: 2 copper layers, 103.8 x 87.8 mm, 19 parts, among them J1 IDC Connector, J2 Mini-DIN-6, J3 Bus_ISA_8bit, Q1 BC547, U1 74LS00, U2 L78L05

Commit message: v1.7.1
- Wrong files upload fix.
Connections:
- J2 pad GND: (no net) -> /GND
Routing:
- net /GND: track 362.4 -> 379.0 mm
Changed lines of the file:
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@@
     (pad "6" thru_hole circle (at 3.35026 11.00074 90) (size 1.3716 1.3716) (drill 0.889) (layers "*.Cu" "*.Mask")
       (net 52 "unconnected-(J2-Pad6)") (pintype "passive+no_connect"))
-    (pad "GND" thru_hole circle (at -6.75894 5.50926 90) (size 4.0005 4.0005) (drill 2.29108) (layers "*.Cu" "*.Mask"))
-    (pad "GND" thru_hole circle (at 0 4.699 90) (size 4.0005 4.0005) (drill 2.29108) (layers "*.Cu" "*.Mask"))
-    (pad "GND" thru_hole circle (at 6.75894 5.50926 90) (size 4.0005 4.0005) (drill 2.29108) (layers "*.Cu" "*.Mask"))
+    (pad "GND" thru_hole circle (at -6.75894 5.50926 90) (size 4.0005 4.0005) (drill 2.29108) (layers "*.Cu" "*.Mask")
+      (net 1 "/GND"))
+    (pad "GND" thru_hole circle (at 0 4.699 90) (size 4.0005 4.0005) (drill 2.29108) (layers "*.Cu" "*.Mask")
+      (net 1 "/GND"))
+    (pad "GND" thru_hole circle (at 6.75894 5.50926 90) (size 4.0005 4.0005) (drill 2.29108) (layers "*.Cu" "*.Mask")
+      (net 1 "/GND"))
     (model "r_mini_dins/minidin_6.wrl"
       (offset (xyz 0 0 0))
@@
   (segment (start 67.31 74.93) (end 67.31 72.39) (width 0.8) (layer "B.Cu") (net 1))
   (segment (start 67.31 72.39) (end 73.66 72.39) (width 0.8) (layer "B.Cu") (net 1))
+  (segment (start 108.76026 30.12186) (end 111.76 27.12212) (width 0.8) (layer "B.Cu") (net 1))
   (segment (start 57.15 69.85) (end 59.69 72.39) (width 0.8) (layer "B.Cu") (net 1))
   (segment (start 108.76026 24.12238) (end 108.76026 30.5308) (width 0.8) (layer "B.Cu") (net 1))
   (segment (start 111.76 50.8) (end 111.76 73.66) (width 0.8) (layer "B.Cu") (net 1))
   (segment (start 92.71 76.2) (end 90.17 73.66) (width 0.8) (layer "B.Cu") (net 1))
+  (segment (start 111.76 27.12212) (end 111.76 33.0708) (width 0.8) (layer "B.Cu") (net 1))
   (segment (start 36.83 20.32) (end 25.4 31.75) (width 0.8) (layer "B.Cu") (net 1))
   (segment (start 59.69 72.39) (end 67.31 72.39) (width 0.8) (layer "B.Cu") (net 1))
@@
   (segment (start 73.66 72.39) (end 74.93 72.39) (width 0.8) (layer "B.Cu") (net 1))
   (segment (start 87.63 76.2) (end 90.17 73.66) (width 0.8) (layer "B.Cu") (net 1))
+  (segment (start 112.57026 33.88106) (end 112.57026 39.82974) (width 0.8) (layer "B.Cu") (net 1))
   (segment (start 74.93 72.39) (end 78.74 76.2) (width 0.8) (layer "B.Cu") (net 1))
   (segment (start 90.17 73.66) (end 90.17 63.5) (width 0.8) (layer "B.Cu") (net 1))
@@
   (segment (start 71.12 78.74) (end 67.31 74.93) (width 0.8) (layer "B.Cu") (net 1))
   (segment (start 109.22 76.2) (end 106.68 76.2) (width 0.8) (layer "B.Cu") (net 1))
+  (segment (start 108.76026 30.5308) (end 108.76026 30.12186) (width 0.8) (layer "B.Cu") (net 1))
   (segment (start 55.88 52.07) (end 57.15 50.8) (width 0.8) (layer "B.Cu") (net 1))
   (segment (start 91.44 86.36) (end 83.82 78.74) (width 0.8) (layer "B.Cu") (net 1))
