File: schematics/In_a_Box/KiCad_Project/ps2_mouse_to_serial_port_adapter_in_a_box.kicad_sch (KiCad schematic)
At the start: 24 parts, among them J1 DC IN, J2 PS/2 & USB, J3 Serial Port, Q1 BC547, SW1 Switch ON/OFF, U1 74LS00, U2 L78L05, U3 L7805

Commit message: v1.5.0
- Ajustadas las placas "Stand alone" y "In-a-box" al tamaño standard de
  90x70 mm.
- Añadidas a estas placas las zonas de relleno a masa (GND).
- Añadidas las serigrafias con los valores de todos los componentes en todas
  las versiones de las placas.
Connections:
- net +5V: now reaches A1.30 (VIN), C1.1, C4.1, C5.1, C6.1, J2.7 (Pin_7), J2.8 (Pin_8), R3.1, R5.1, U1.14 (VCC), U3.3 (OUT)
- net GND: now reaches A1.29 (GND), C1.2, C2.2, C3.2, C4.2, C5.2, C6.2, D3.1 (K), D4.1 (K), J1.2 (Pin_2), J2.1 (Pin_1), J2.2 (Pin_2), J3.1 (Pin_1), Q1.3 (E), R2.2, U1.7 (GND), U2.2 (GND), U3.2 (GND)
Changed lines of the file:
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@@
   (title_block
     (title "PS/2 Mouse to Serial Port Adapter")
-    (date "2023-08-12")
-    (rev "3")
+    (date "2023-08-13")
+    (rev "4")
     (company "Cesar Rincon")
     (comment 1 "NightFox & Co.")
@@
     (effects (font (size 1.27 1.27)) (justify left bottom))
   )
-  (text "GND" (at 151.13 187.96 0)
-    (effects (font (size 1.27 1.27)) (justify left bottom))
-  )
   (text "GND" (at 16.51 157.48 0)
     (effects (font (size 1.27 1.27)) (justify left bottom))
@@
     (effects (font (size 1.27 1.27)) (justify left bottom))
   )
+  (label "+5V" (at 262.89 25.4 0) (fields_autoplaced)
+    (effects (font (size 1.27 1.27)) (justify left bottom))
+  )
+  (label "GND" (at 152.4 184.15 0) (fields_autoplaced)
+    (effects (font (size 1.27 1.27)) (justify left bottom))
+  )

Commit message: v1.5.1
- Arreglada la serigrafía del conector MINI-DIN-6 (PS/2), la cual se superponía en algunas zonas de soldado.
- En todas las placas se añade el símbolo de los agujeros de montaje con el tamaño estándar M3.
Parts:
- added H1, H2, H3, H4: MountingHole, MountingHole:MountingHole_3.2mm_M3, symbol Mechanical:MountingHole
Changed lines of the file:
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@@
   (title_block
     (title "PS/2 Mouse to Serial Port Adapter")
-    (date "2023-08-13")
-    (rev "4")
+    (date "2023-08-14")
+    (rev "5")
     (company "Cesar Rincon")
     (comment 1 "NightFox & Co.")
@@
     (effects (font (size 1.27 1.27)) (justify left bottom))
   )
+  (symbol (lib_id "Mechanical:MountingHole") (at -86.36 71.12 0) (unit 1)
+    (in_bom yes) (on_board yes) (dnp no) (fields_autoplaced)
+    (property "Reference" "H3" (at -83.82 69.85 0)
+      (effects (font (size 1.27 1.27)) (justify left))
+    )
+    (property "Value" "MountingHole" (at -83.82 72.39 0)
+      (effects (font (size 1.27 1.27)) (justify left))
+    )
+    (property "Footprint" "MountingHole:MountingHole_3.2mm_M3" (at -86.36 71.12 0)
+      (effects (font (size 1.27 1.27)) hide)
+    )
+    (property "Datasheet" "~" (at -86.36 71.12 0)
+      (effects (font (size 1.27 1.27)) hide)
+    )
+    (instances
+      (project "ps2_mouse_to_serial_port_adapter_in_a_box"
+        (path "/a7ffaf24-5f7f-4c3c-9493-bf517f6435f3"
+          (reference "H3") (unit 1)
+        )
+      )
+    )
+  )
   (symbol (lib_id "Device:C") (at 243.84 45.72 0) (unit 1)
     (in_bom yes) (on_board yes) (dnp no) (fields_autoplaced)
@@
     )
   )
+  (symbol (lib_id "Mechanical:MountingHole") (at -86.36 66.04 0) (unit 1)
+    (in_bom yes) (on_board yes) (dnp no) (fields_autoplaced)
+    (property "Reference" "H2" (at -83.82 64.77 0)
+      (effects (font (size 1.27 1.27)) (justify left))
+    )
+    (property "Value" "MountingHole" (at -83.82 67.31 0)
+      (effects (font (size 1.27 1.27)) (justify left))
+    )
+    (property "Footprint" "MountingHole:MountingHole_3.2mm_M3" (at -86.36 66.04 0)
+      (effects (font (size 1.27 1.27)) hide)
+    )
+    (property "Datasheet" "~" (at -86.36 66.04 0)
+      (effects (font (size 1.27 1.27)) hide)
+    )
+    (instances
+      (project "ps2_mouse_to_serial_port_adapter_in_a_box"
+        (path "/a7ffaf24-5f7f-4c3c-9493-bf517f6435f3"
+          (reference "H2") (unit 1)
+        )
+      )
+    )
+  )
+  (symbol (lib_id "Mechanical:MountingHole") (at -86.36 76.2 0) (unit 1)
+    (in_bom yes) (on_board yes) (dnp no) (fields_autoplaced)
+    (property "Reference" "H4" (at -83.82 74.93 0)
+      (effects (font (size 1.27 1.27)) (justify left))
+    )
+    (property "Value" "MountingHole" (at -83.82 77.47 0)
+      (effects (font (size 1.27 1.27)) (justify left))
+    )
+    (property "Footprint" "MountingHole:MountingHole_3.2mm_M3" (at -86.36 76.2 0)
+      (effects (font (size 1.27 1.27)) hide)
+    )
+    (property "Datasheet" "~" (at -86.36 76.2 0)
+      (effects (font (size 1.27 1.27)) hide)
+    )
+    (instances
+      (project "ps2_mouse_to_serial_port_adapter_in_a_box"
+        (path "/a7ffaf24-5f7f-4c3c-9493-bf517f6435f3"
+          (reference "H4") (unit 1)
+        )
+      )
+    )
+  )
   (symbol (lib_id "Connector:Conn_01x03_Pin") (at 22.86 158.75 0) (unit 1)
     (in_bom yes) (on_board yes) (dnp no)
@@
         )
       )
+    )
+  )
+  (symbol (lib_id "Mechanical:MountingHole") (at -86.36 60.96 0) (unit 1)
+    (in_bom yes) (on_board yes) (dnp no) (fields_autoplaced)
+    (property "Reference" "H1" (at -83.82 59.69 0)
+      (effects (font (size 1.27 1.27)) (justify left))
+    )
+    (property "Value" "MountingHole" (at -83.82 62.23 0)
+      (effects (font (size 1.27 1.27)) (justify left))
+    )
+    (property "Footprint" "MountingHole:MountingHole_3.2mm_M3" (at -86.36 60.96 0)
+      (effects (font (size 1.27 1.27)) hide)
+    )
+    (property "Datasheet" "~" (at -86.36 60.96 0)
+      (effects (font (size 1.27 1.27)) hide)
+    )
+    (instances
+      (project "ps2_mouse_to_serial_port_adapter_in_a_box"
+        (path "/a7ffaf24-5f7f-4c3c-9493-bf517f6435f3"
+          (reference "H1") (unit 1)
+        )
+      )

Commit message: v1.7.0
- Modificadas las huellas de todas las placas para que los componentes TO92 resulten más fáciles de soldar a mano.
- Modificadas las conexiones del conector IDC en la placa ISA para poder usar un cable IDC a DB9 comercial, sin necesidad de realizarle modificaciones.
- Añadido el modelo en formato FreeCad y el archivo STL del soporte para la placa ISA. Estos archivos estan preparados para poder realizar la impresión en 3D del soporte. Se recomienda un in-fill del 100%.
Parts:
- Q1, U2: footprint Package_TO_SOT_THT:TO-92_Inline -> Package_TO_SOT_THT:TO-92_HandSolder
- U1: footprint (none) -> Package_DIP:DIP-14_W7.62mm_Socket
Changed lines of the file:
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@@
   (title_block
     (title "PS/2 Mouse to Serial Port Adapter")
-    (date "2023-08-14")
-    (rev "5")
+    (date "2023-08-28")
+    (rev "6")
     (company "Cesar Rincon")
     (comment 1 "NightFox & Co.")
@@
       (effects (font (size 1.27 1.27)))
     )
-    (property "Footprint" "" (at -81.28 35.56 0)
+    (property "Footprint" "Package_DIP:DIP-14_W7.62mm_Socket" (at -81.28 35.56 0)
       (effects (font (size 1.27 1.27)) hide)
     )
@@
       (effects (font (size 1.27 1.27)) (justify left))
     )
-    (property "Footprint" "Package_TO_SOT_THT:TO-92_Inline" (at 134.62 160.655 0)
+    (property "Footprint" "Package_TO_SOT_THT:TO-92_HandSolder" (at 134.62 160.655 0)
       (effects (font (size 1.27 1.27) italic) (justify left) hide)
     )
@@
       (effects (font (size 1.27 1.27)))
     )
-    (property "Footprint" "Package_TO_SOT_THT:TO-92_Inline" (at 86.36 153.035 0)
+    (property "Footprint" "Package_TO_SOT_THT:TO-92_HandSolder" (at 86.36 153.035 0)
       (effects (font (size 1.27 1.27) italic) hide)
     )
@@
       (effects (font (size 1.27 1.27)))
     )
-    (property "Footprint" "" (at -81.28 10.16 0)
-      (effects (font (size 1.27 1.27)) hide)
-    )
+    (property "Footprint" "Package_DIP:DIP-14_W7.62mm_Socket" (at -81.28 10.16 0)
+      (effects (font (size 1.27 1.27)) hide)
+    )
